Commit message: fix link for kinect

File: map_bot/urdf/map_bot.xacro (robot description, xacro)
@@ -32,4 +32,5 @@
   <xacro:property name="wheel_length" value="0.05" />
   <xacro:property name="wheel_radius" value="0.1" />
+  <xacro:property name="pi" value="3.14159" />
   <xacro:include filename="$(find map_bot)/urdf/map_bot.gazebo" />
   <link name="robot_footprint"></link>
@@ -145,5 +146,5 @@
   </joint>
   <!-- Sensor: Camera -->
-  <link name="camera">
+  <link name="camera_link">
     <inertial>
       <origin xyz="0 0 0" rpy="0 0 0"/>
@@ -168,6 +169,13 @@
     <origin xyz="${base_x_size / 2.0} 0 0" rpy="0 0 0"/>
     <parent link="chassis"/>
-    <child link="camera"/>
-  </joint>>
+    <child link="camera_link"/>
+  </joint>
+  <joint name="camera_optical_joint" type="fixed">
+    <origin xyz="0.0 0.0 0.0" rpy="${-pi/2} 0 ${-pi/2}"/>
+    <parent link="camera_link"/>
+    <child link="camera_link_optical"/>
+  </joint>
+  <link name="camera_link_optical">
+  </link>
   <!-- Sensor: Laser RangeFinder -->
   <link name="hokuyo">
